File: unicorne-cherry-mx-3x5-reversible/unicorne-cherry-mx-3x5-reversible.kicad_pcb (KiCad board)
At the start: 2 copper layers, 114.7 x 91.4 mm, 84 parts, among them J1 MJ-4PP-9, J2 Nice!View, J3 Conn_01x02, J4 Conn_01x03, SW1 SW_MX_HS, SW10 SW_MX_HS, SW11 SW_MX_HS, SW12 SW_MX_HS, SW13 SW_MX_HS, SW14 SW_MX_HS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

Commit message: hardware handedness
Parts:
- added JP9: Jumper_3_Bridged12, TB2086_MISC:SolderJumper-3_P1.3mm_Bridged2Bar12_RoundedPad1.0x1.5mm_rev, F.Cu at (189.0, 110.4)
- added R3: 4.7k, TB2086_SMD:R_0805_2012Metric_Pad1.20x1.40mm_HandSolder_rev, F.Cu at (185.3, 109.4)
- added R4: 4.7k, TB2086_SMD:R_0805_2012Metric_Pad1.20x1.40mm_HandSolder_rev, F.Cu at (185.3, 111.3)
- D1, D10, D11, D12, D13, D14, D15, D16, D17, D18, D2, D3, D4, D5, D6, D7, D8, D9: footprint KBD_PARTS:D3_SMD_rev -> TB2086_SMD:D3_SMD_rev
- H1, H2: footprint KBD_PARTS:M2_Hole_TH -> TB2086_MISC:M2_Hole_TH
- H3, H4, H5, H6, H7: footprint KBD_PARTS:M2_Hole_TH_Outside -> TB2086_MISC:M2_Hole_TH_Outside
- J1: footprint KBD_PARTS:TRRS-PJ-320A-rev -> TB2086_MISC:TRRS-PJ-320A-rev
- J2: footprint KBD_PARTS:Nice!View -> TB2086_MISC:Nice!View
- J3: footprint KBD_PARTS:Molex_Pico-EZmate_78171-0002_1x02-1MP_P1.20mm_Vertical_rev -> TB2086_SMD:Molex_Pico-EZmate_78171-0002_1x02-1MP_P1.20mm_Vertical_rev
- J4: footprint KBD_PARTS:StripLED_rev -> TB2086_MISC:StripLED_rev
- L1, L10, L11, L12, L13, L14, L15, L16, L17, L18, L2, L3, L4, L5, L6, L7, L8, L9: value SK6812MINI -> SK6812MINI-E; footprint KBD_PARTS:LED_SK6812MINI_PLCC4_3.5x3.5mm_P1.75mm_back_rev -> TB2086_LED:LED_SK6812MINI-E_rev
- L19, L20, L21, L22, L23, L24: footprint KBD_PARTS:LED_SK6812MINI_PLCC4_3.5x3.5mm_P1.75mm_rev -> TB2086_LED:LED_SK6812MINI_PLCC4_3.5x3.5mm_P1.75mm_rev_all
- PSW1: footprint Akizukidenshi:SW_SPDT_PCM12_reversible -> TB2086_SMD:SW_SPDT_PCM12_reversible
- RSW1: value SW_PUSH -> SMT 2X4X3.5MM Tactile Tact Push Button; footprint KBD_PARTS:SMT 2X4X3.5MM Tactile Tact Push Button -> TB2086_SMD:SMT 2X4X3.5MM Tactile Tact Push Button rev
- SW1, SW10, SW11, SW12, SW13, SW14, SW15, SW16, SW17, SW2, SW3, SW4, SW5, SW6, SW7, SW8, SW9: footprint KBD_PARTS:SW_MX_HS_1u_reversible -> TB2086_KEYSWITCH:SW_MX_HS_1u_reversible
- SW18: footprint KBD_PARTS:SW_MX_HS_1.5u_reversible -> TB2086_KEYSWITCH:SW_MX_HS_1u_reversible
- U1: footprint KBD_PARTS:ProMicro-ish-rev-unrouted_3x5 -> TB2086_MISC:ProMicro-ish-dn-rev-unrouted_3x5
- moved H6 0.13 mm to (98.5, 105.8)
- moved H7 0.13 mm to (98.5, 86.8)
- turned L14 to 0 degrees
- turned L17 to 165 degrees
- turned L19 to 180 degrees
- turned L20 to 180 degrees
- turned L21 to 180 degrees
- turned L5 to 180 degrees
- turned L6 to 0 degrees
- turned L9 to 0 degrees
Connections:
- J1 pad A: unconnected-(J1-PadA) -> SCL
- J1 pad B: DATA -> Net-(JP9-C)
- L1 pad 1: unconnected-(L1-DOUT-Pad1) -> VCC
- L1 pad 2: GND -> unconnected-(L1-DOUT-Pad2)
- L1 pad 3: Net-(L1-DIN) -> GND
- L1 pad 4: VCC -> Net-(L1-DIN)
- L10 pad 1: Net-(L10-DOUT) -> VCC
- L10 pad 2: GND -> Net-(L10-DOUT)
- L10 pad 3: Net-(L10-DIN) -> GND
- L10 pad 4: VCC -> Net-(L10-DIN)
- L11 pad 1: Net-(L11-DOUT) -> VCC
- L11 pad 2: GND -> Net-(L11-DOUT)
- L11 pad 3: Net-(L11-DIN) -> GND
- L11 pad 4: VCC -> Net-(L11-DIN)
- L12 pad 1: Net-(L11-DIN) -> VCC
- L12 pad 2: GND -> Net-(L11-DIN)
- L12 pad 3: Net-(L12-DIN) -> GND
- L12 pad 4: VCC -> Net-(L12-DIN)
- L13 pad 1: Net-(L13-DOUT) -> VCC
- L13 pad 2: GND -> Net-(L13-DOUT)
- L13 pad 3: Net-(L13-DIN) -> GND
- L13 pad 4: VCC -> Net-(L13-DIN)
- L14 pad 1: Net-(L14-DOUT) -> VCC
- L14 pad 2: GND -> Net-(L14-DOUT)
- L14 pad 3: Net-(L14-DIN) -> GND
- L14 pad 4: VCC -> Net-(L14-DIN)
- L15 pad 1: Net-(L10-DIN) -> VCC
- L15 pad 2: GND -> Net-(L10-DIN)
- L15 pad 3: Net-(L15-DIN) -> GND
- L15 pad 4: VCC -> Net-(L15-DIN)
- L16 pad 1: Net-(L13-DIN) -> VCC
- L16 pad 2: GND -> Net-(L13-DIN)
- L16 pad 3: Net-(L16-DIN) -> GND
- L16 pad 4: VCC -> Net-(L16-DIN)
- L17 pad 1: Net-(L16-DIN) -> VCC
- L17 pad 2: GND -> Net-(L16-DIN)
- L17 pad 3: Net-(L14-DOUT) -> GND
- L17 pad 4: VCC -> Net-(L14-DOUT)
- L18 pad 1: Net-(L15-DIN) -> VCC
- L18 pad 2: GND -> Net-(L15-DIN)
- L18 pad 3: Net-(L18-DIN) -> GND
- L18 pad 4: VCC -> Net-(L18-DIN)
- L2 pad 1: Net-(L2-DOUT) -> VCC
- L2 pad 2: GND -> Net-(L2-DOUT)
- L2 pad 3: Net-(L2-DIN) -> GND
- L2 pad 4: VCC -> Net-(L2-DIN)
- L3 pad 1: Net-(L2-DIN) -> VCC
- L3 pad 2: GND -> Net-(L2-DIN)
- L3 pad 3: Net-(L3-DIN) -> GND
- L3 pad 4: VCC -> Net-(L3-DIN)
- L4 pad 1: Net-(L4-DOUT) -> VCC
- L4 pad 2: GND -> Net-(L4-DOUT)
- L4 pad 3: Net-(L4-DIN) -> GND
- L4 pad 4: VCC -> Net-(L4-DIN)
- L5 pad 1: Net-(L4-DIN) -> VCC
- L5 pad 2: GND -> Net-(L4-DIN)
- L5 pad 3: Net-(L10-DOUT) -> GND
- L5 pad 4: VCC -> Net-(L10-DOUT)
- L6 pad 1: Net-(L1-DIN) -> VCC
- L6 pad 2: GND -> Net-(L1-DIN)
- L6 pad 3: Net-(L11-DOUT) -> GND
- L6 pad 4: VCC -> Net-(L11-DOUT)
- L7 pad 1: Net-(L12-DIN) -> VCC
- L7 pad 2: GND -> Net-(L12-DIN)
- L7 pad 3: Net-(L2-DOUT) -> GND
- L7 pad 4: VCC -> Net-(L2-DOUT)
- L8 pad 1: Net-(L3-DIN) -> VCC
- L8 pad 2: GND -> Net-(L3-DIN)
- L8 pad 3: Net-(L13-DOUT) -> GND
- L8 pad 4: VCC -> Net-(L13-DOUT)
- L9 pad 1: Net-(L14-DIN) -> VCC
- L9 pad 2: GND -> Net-(L14-DIN)
- L9 pad 3: Net-(L4-DOUT) -> GND
- L9 pad 4: VCC -> Net-(L4-DOUT)
Routing:
- net VCC: track 562.3 -> 530.0 mm, vias 3 -> 2
- net SCL: track 39.2 -> 62.4 mm, vias 2 -> 4
- net GND: track 57.7 -> 34.8 mm, vias 21 -> 13
- net Net-(JP9-C): track 0.00 -> 17.6 mm
- net Net-(L13-DIN): track 38.9 -> 25.8 mm
- net DATA: track 77.8 -> 64.8 mm, vias 1 -> 2
- net SDA: track 61.7 -> 73.7 mm, vias 2 -> 4
- net col2: track 178.6 -> 167.2 mm
- net Net-(L18-DIN): track 46.5 -> 35.1 mm, vias 0 -> 2
- net Net-(L16-DIN): track 15.3 -> 25.5 mm
- net Net-(L22-DOUT): track 47.9 -> 57.7 mm
- net Net-(L20-DIN): track 52.4 -> 44.1 mm
- net Net-(L14-DOUT): track 28.9 -> 37.0 mm
- net Net-(L10-DOUT): track 28.0 -> 19.9 mm, vias 0 -> 1
- net Net-(L14-DIN): track 24.5 -> 31.3 mm
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Other:
- board text added: "Left Up"
- board text added: "Right Up"
- board text removed: "left"
- board text removed: "right"

Commit message: small tweak
Routing:
- net Net-(JP9-C): track 17.6 -> 14.8 mm
- net SCL: track 62.4 -> 60.3 mm
- net SDA: track 73.7 -> 72.5 mm
- net VCC: track 530.0 -> 529.3 mm
- net col2: track 167.2 -> 166.6 mm
- net GND: vias 13 -> 12
Other:
- outline, holes or cut-outs redrawn
- board text added: "left hand"
- board text added: "right hand"
- board text removed: "Left Up"
- board text removed: "Right Up"
