File: unicorne-hybrid-mx-3x5-reversible/unicorne-hybrid-mx-3x5-reversible.kicad_pcb (KiCad board)
At the start: 2 copper layers, 114.7 x 91.4 mm, 84 parts, among them J1 MJ-4PP-9, J2 Nice!View, J3 Conn_01x02, J4 Conn_01x03, SW1 SW_MX_HS, SW10 SW_MX_HS, SW11 SW_MX_HS, SW12 SW_MX_HS, SW13 SW_MX_HS, SW14 SW_MX_HS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

Commit message: hybrid
Parts:
- SW16, SW17: value SW_MX_HS -> SW_CHOC_HS; footprint KBD_PARTS:SW_MX_HS_1u_reversible -> KBD_PARTS:SW_choc_v1_v2_HS_1u_reversible
- SW18: value SW_MX_HS -> SW_CHOC_HS; footprint KBD_PARTS:SW_MX_HS_1.5u_reversible -> KBD_PARTS:SW_choc_v1_v2_HS_1u_reversible
- moved D17 18.1 mm to (150.3, 126.6), turned to -105 degrees
- moved L16 10.00 mm to (136.8, 125.7)
- moved L18 9.97 mm to (175.3, 134.2)
- moved L17 9.79 mm to (158.8, 128.2)
- moved D18 8.07 mm to (178.9, 126.6), turned to -30 degrees
- moved D16 6.85 mm to (145.3, 126.3), turned to -90 degrees
Routing:
- net VCC: track 562.3 -> 524.1 mm
- net row3: track 115.6 -> 89.2 mm, vias 1 -> 3
- net col2: track 178.6 -> 201.1 mm, vias 1 -> 2
- net col4: track 130.5 -> 148.1 mm
- net Net-(L13-DIN): track 38.9 -> 23.2 mm
- net Net-(L18-DIN): track 46.5 -> 30.9 mm
- net Net-(L15-DIN): track 32.6 -> 18.7 mm
- net col3: track 140.9 -> 153.5 mm
- net Net-(D17-A): track 2.46 -> 13.9 mm
- net Net-(L14-DOUT): track 28.9 -> 18.4 mm
- net Net-(D16-A): track 3.92 -> 12.5 mm
- net Net-(D18-A): track 5.85 -> 14.0 mm
- net Net-(L16-DIN): track 15.3 -> 17.6 mm

Commit message: hardware handedness
Parts:
- added JP9: Jumper_3_Bridged12, TB2086_MISC:SolderJumper-3_P1.3mm_Bridged2Bar12_RoundedPad1.0x1.5mm_rev, F.Cu at (189.3, 110.2)
- added R3: 4.7k, TB2086_SMD:R_0805_2012Metric_Pad1.20x1.40mm_HandSolder_rev, F.Cu at (185.8, 109.1)
- added R4: 4.7k, TB2086_SMD:R_0805_2012Metric_Pad1.20x1.40mm_HandSolder_rev, F.Cu at (185.8, 111.0)
- D1, D10, D11, D12, D13, D14, D15, D16, D17, D18, D2, D3, D4, D5, D6, D7, D8, D9: footprint KBD_PARTS:D3_SMD_rev -> TB2086_SMD:D3_SMD_rev
- H1, H2: footprint KBD_PARTS:M2_Hole_TH -> TB2086_MISC:M2_Hole_TH
- H3, H4, H5, H6, H7: footprint KBD_PARTS:M2_Hole_TH_Outside -> TB2086_MISC:M2_Hole_TH_Outside
- J1: footprint KBD_PARTS:TRRS-PJ-320A-rev -> TB2086_MISC:TRRS-PJ-320A-rev
- J2: footprint KBD_PARTS:Nice!View -> TB2086_MISC:Nice!View
- J4: footprint KBD_PARTS:StripLED_rev -> TB2086_MISC:StripLED_rev
- JP1, JP2, JP3, JP4, JP5, JP6, JP7, JP8: footprint Jumper:SolderJumper-2_P1.3mm_Open_TrianglePad1.0x1.5mm -> TB2086_MISC:SolderJumper-2_P1.3mm_Open_TrianglePad1.0x1.5mm
- L1, L10, L11, L12, L13, L14, L15, L16, L17, L18, L2, L3, L4, L5, L6, L7, L8, L9: value SK6812MINI -> SK6812MINI-E; footprint KBD_PARTS:LED_SK6812MINI_PLCC4_3.5x3.5mm_P1.75mm_back_rev -> TB2086_LED:LED_SK6812MINI-E_rev
- L19, L20, L21, L22, L23, L24: footprint KBD_PARTS:LED_SK6812MINI_PLCC4_3.5x3.5mm_P1.75mm_rev -> TB2086_LED:LED_SK6812MINI_PLCC4_3.5x3.5mm_P1.75mm_rev_all
- PSW1: footprint Akizukidenshi:SW_SPDT_PCM12_reversible -> TB2086_SMD:SW_SPDT_PCM12_reversible
- RSW1: footprint KBD_PARTS:SMT 2X4X3.5MM Tactile Tact Push Button -> TB2086_SMD:SMT 2X4X3.5MM Tactile Tact Push Button rev
- SW1, SW10, SW11, SW12, SW13, SW14, SW15, SW2, SW3, SW4, SW5, SW6, SW7, SW8, SW9: footprint KBD_PARTS:SW_MX_HS_1u_reversible -> TB2086_KEYSWITCH:SW_MX_HS_1u_reversible
- SW16, SW17: footprint KBD_PARTS:SW_choc_v1_v2_HS_1u_reversible -> TB2086_KEYSWITCH:SW_choc_v1_v2_HS_1u_reversible
- SW18: footprint KBD_PARTS:SW_choc_v1_v2_HS_1u_reversible -> TB2086_KEYSWITCH:SW_choc_v1_v2_HS_1.5u_reversible
- U1: footprint KBD_PARTS:ProMicro-ish-rev-unrouted_3x5 -> TB2086_MISC:ProMicro-ish-dn-rev-unrouted_3x5
- moved H6 0.13 mm to (98.5, 105.8)
- moved H7 0.13 mm to (98.5, 86.8)
- turned L11 to 180 degrees
- turned L13 to 180 degrees
- turned L5 to 180 degrees
- turned L8 to 180 degrees
Connections:
- J1 pad A: unconnected-(J1-PadA) -> SCL
- J1 pad B: DATA -> Net-(JP9-C)
- L1 pad 1: unconnected-(L1-DOUT-Pad1) -> VCC
- L1 pad 2: GND -> unconnected-(L1-DOUT-Pad2)
- L1 pad 3: Net-(L1-DIN) -> GND
- L1 pad 4: VCC -> Net-(L1-DIN)
- L10 pad 1: Net-(L10-DOUT) -> VCC
- L10 pad 2: GND -> Net-(L10-DOUT)
- L10 pad 3: Net-(L10-DIN) -> GND
- L10 pad 4: VCC -> Net-(L10-DIN)
- L11 pad 1: Net-(L11-DOUT) -> VCC
- L11 pad 2: GND -> Net-(L11-DOUT)
- L11 pad 3: Net-(L11-DIN) -> GND
- L11 pad 4: VCC -> Net-(L11-DIN)
- L12 pad 1: Net-(L11-DIN) -> VCC
- L12 pad 2: GND -> Net-(L11-DIN)
- L12 pad 3: Net-(L12-DIN) -> GND
- L12 pad 4: VCC -> Net-(L12-DIN)
- L13 pad 1: Net-(L13-DOUT) -> VCC
- L13 pad 2: GND -> Net-(L13-DOUT)
- L13 pad 3: Net-(L13-DIN) -> GND
- L13 pad 4: VCC -> Net-(L13-DIN)
- L14 pad 1: Net-(L14-DOUT) -> VCC
- L14 pad 2: GND -> Net-(L14-DOUT)
- L14 pad 3: Net-(L14-DIN) -> GND
- L14 pad 4: VCC -> Net-(L14-DIN)
- L15 pad 1: Net-(L10-DIN) -> VCC
- L15 pad 2: GND -> Net-(L10-DIN)
- L15 pad 3: Net-(L15-DIN) -> GND
- L15 pad 4: VCC -> Net-(L15-DIN)
- L16 pad 1: Net-(L13-DIN) -> VCC
- L16 pad 2: GND -> Net-(L13-DIN)
- L16 pad 3: Net-(L16-DIN) -> GND
- L16 pad 4: VCC -> Net-(L16-DIN)
- L17 pad 1: Net-(L16-DIN) -> VCC
- L17 pad 2: GND -> Net-(L16-DIN)
- L17 pad 3: Net-(L14-DOUT) -> GND
- L17 pad 4: VCC -> Net-(L14-DOUT)
- L18 pad 1: Net-(L15-DIN) -> VCC
- L18 pad 2: GND -> Net-(L15-DIN)
- L18 pad 3: Net-(L18-DIN) -> GND
- L18 pad 4: VCC -> Net-(L18-DIN)
- L2 pad 1: Net-(L2-DOUT) -> VCC
- L2 pad 2: GND -> Net-(L2-DOUT)
- L2 pad 3: Net-(L2-DIN) -> GND
- L2 pad 4: VCC -> Net-(L2-DIN)
- L3 pad 1: Net-(L2-DIN) -> VCC
- L3 pad 2: GND -> Net-(L2-DIN)
- L3 pad 3: Net-(L3-DIN) -> GND
- L3 pad 4: VCC -> Net-(L3-DIN)
- L4 pad 1: Net-(L4-DOUT) -> VCC
- L4 pad 2: GND -> Net-(L4-DOUT)
- L4 pad 3: Net-(L4-DIN) -> GND
- L4 pad 4: VCC -> Net-(L4-DIN)
- L5 pad 1: Net-(L4-DIN) -> VCC
- L5 pad 2: GND -> Net-(L4-DIN)
- L5 pad 3: Net-(L10-DOUT) -> GND
- L5 pad 4: VCC -> Net-(L10-DOUT)
- L6 pad 1: Net-(L1-DIN) -> VCC
- L6 pad 2: GND -> Net-(L1-DIN)
- L6 pad 3: Net-(L11-DOUT) -> GND
- L6 pad 4: VCC -> Net-(L11-DOUT)
- L7 pad 1: Net-(L12-DIN) -> VCC
- L7 pad 2: GND -> Net-(L12-DIN)
- L7 pad 3: Net-(L2-DOUT) -> GND
- L7 pad 4: VCC -> Net-(L2-DOUT)
- L8 pad 1: Net-(L3-DIN) -> VCC
- L8 pad 2: GND -> Net-(L3-DIN)
- L8 pad 3: Net-(L13-DOUT) -> GND
- L8 pad 4: VCC -> Net-(L13-DOUT)
- L9 pad 1: Net-(L14-DIN) -> VCC
- L9 pad 2: GND -> Net-(L14-DIN)
- L9 pad 3: Net-(L4-DOUT) -> GND
- L9 pad 4: VCC -> Net-(L4-DOUT)
Routing:
- net Net-(L3-DIN): track 33.0 -> 56.2 mm, vias 1 -> 0
- net GND: track 57.7 -> 34.9 mm, vias 21 -> 17
- net SCL: track 39.2 -> 61.8 mm, vias 2 -> 4
- net VCC: track 524.1 -> 505.1 mm
- net col2: track 201.1 -> 184.9 mm, vias 2 -> 1
- net Net-(JP9-C): track 0.00 -> 16.1 mm
- net DATA: track 77.6 -> 64.7 mm, vias 1 -> 2
- net Net-(L14-DOUT): track 18.4 -> 29.9 mm
- net SDA: track 61.7 -> 73.2 mm, vias 2 -> 4
- net Net-(L22-DOUT): track 47.9 -> 57.1 mm
- net Net-(L11-DIN): track 16.0 -> 23.1 mm
- net Net-(L4-DIN): track 15.4 -> 21.5 mm
- net Net-(L10-DIN): track 28.4 -> 22.5 mm
- net Net-(L11-DOUT): track 25.9 -> 20.4 mm
- net Net-(L1-DIN): track 26.9 -> 21.5 mm
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
Commit message: small tweak
Parts:
- moved R3 0.20 mm to (185.8, 109.3)
- moved R4 0.20 mm to (185.8, 111.2)
- moved JP9 0.20 mm to (189.3, 110.4)
Routing:
- net VCC: track 505.1 -> 499.8 mm
- net SCL: track 61.8 -> 59.5 mm
- net SDA: track 73.2 -> 71.4 mm
- net Net-(JP9-C): track 16.1 -> 15.4 mm
- net GND: vias 17 -> 16
Other:
- outline, holes or cut-outs redrawn
- board text added: "left hand"
- board text added: "right hand"
- board text added: "uniCorne Hybrid"
- board text removed: "left"
- board text removed: "right"
- board text removed: "uniCorne Cherry"
