File: unicorne-hybrid-mx-3x5-reversible/unicorne-hybrid-mx-3x5-reversible.kicad_sch (KiCad schematic)
At the start: 84 parts, among them J1 MJ-4PP-9, J2 Nice!View, J3 Conn_01x02, J3 Conn_01x03, SW1 SW_MX_HS, SW10 SW_MX_HS, SW11 SW_MX_HS, SW12 SW_MX_HS, SW13 SW_MX_HS, SW14 SW_MX_HS, SW15 SW_MX_HS, SW16 SW_CHOC_HS, SW17 SW_CHOC_HS, SW18 SW_CHOC_HS, SW2 SW_MX_HS, SW3 SW_MX_HS, SW4 SW_MX_HS, SW5 SW_MX_HS, SW6 SW_MX_HS, SW7 SW_MX_HS, SW8 SW_MX_HS, SW9 SW_MX_HS, U1 ProMicro-ish

Commit message: hardware handedness
Parts:
- removed J1: MJ-4PP-9, KBD_PARTS:TRRS-PJ-320A-rev, symbol KBD_PARTS:MJ-4PP-9
- added J1: MJ-4PP-9, TB2086_MISC:TRRS-PJ-320A-rev, symbol TB2086_MISC:MJ-4PP-9
- added JP9: Jumper_3_Bridged12, TB2086_MISC:SolderJumper-3_P1.3mm_Bridged2Bar12_RoundedPad1.0x1.5mm_rev, symbol Jumper:Jumper_3_Bridged12
- added R3, R4: 4.7k, TB2086_SMD:R_0805_2012Metric_Pad1.20x1.40mm_HandSolder_rev, symbol Device:R
- D10, D11, D12, D14, D15, D16, D17, D18, D19, D2, D20, D21, D3, D4, D5, D6, D8, D9: footprint KBD_PARTS:D3_SMD_rev -> TB2086_SMD:D3_SMD_rev
- H1, H2: footprint KBD_PARTS:M2_Hole_TH -> TB2086_MISC:M2_Hole_TH
- H3, H4, H5, H6, H7: footprint KBD_PARTS:M2_Hole_TH_Outside -> TB2086_MISC:M2_Hole_TH_Outside
- J2: footprint KBD_PARTS:Nice!View -> TB2086_MISC:Nice!View
- J3: footprint KBD_PARTS:StripLED_rev -> TB2086_MISC:StripLED_rev
- JP2, JP4, JP5, JP6, JP7, JP9: footprint Jumper:SolderJumper-2_P1.3mm_Open_TrianglePad1.0x1.5mm -> TB2086_MISC:SolderJumper-2_P1.3mm_Open_TrianglePad1.0x1.5mm
- L1, L10, L11, L12, L13, L14, L15, L16, L17, L18, L2, L3, L4, L5, L6, L7, L8, L9: value SK6812MINI -> SK6812MINI-E; footprint KBD_PARTS:LED_SK6812MINI_PLCC4_3.5x3.5mm_P1.75mm_back_rev -> TB2086_LED:LED_SK6812MINI-E_rev; symbol KBD_PARTS:SK6812MINI_back -> TB2086_LED:SK6812MINI-E
- L19, L20, L21, L22, L23, L24: footprint KBD_PARTS:LED_SK6812MINI_PLCC4_3.5x3.5mm_P1.75mm_rev -> TB2086_LED:LED_SK6812MINI_PLCC4_3.5x3.5mm_P1.75mm_rev_all; symbol KBD_PARTS:SK6812MINI -> TB2086_LED:SK6812MINI
- PSW1: footprint Akizukidenshi:SW_SPDT_PCM12_reversible -> TB2086_SMD:SW_SPDT_PCM12_reversible
- RSW1: footprint KBD_PARTS:SMT 2X4X3.5MM Tactile Tact Push Button -> TB2086_SMD:SMT 2X4X3.5MM Tactile Tact Push Button rev; symbol KBD_PARTS:SMT 2X4X3.5MM Tactile Tact Push Button -> TB2086_SMD:SMT 2X4X3.5MM Tactile Tact Push Button
- SW1, SW10, SW11, SW12, SW13, SW14, SW15, SW2, SW3, SW4, SW5, SW6, SW7, SW8, SW9: footprint KBD_PARTS:SW_MX_HS_1u_reversible -> TB2086_KEYSWITCH:SW_MX_HS_1u_reversible; symbol KBD_PARTS:SW_MX_HS -> TB2086_KEYSWITCH:SW_MX_HS
- SW16, SW17: footprint KBD_PARTS:SW_choc_v1_v2_HS_1u_reversible -> TB2086_KEYSWITCH:SW_choc_v1_v2_HS_1u_reversible; symbol KBD_PARTS:SW_CHOC_HS -> TB2086_KEYSWITCH:SW_CHOC_HS
- SW18: footprint KBD_PARTS:SW_choc_v1_v2_HS_1u_reversible -> TB2086_KEYSWITCH:SW_choc_v1_v2_HS_1.5u_reversible; symbol KBD_PARTS:SW_CHOC_HS -> TB2086_KEYSWITCH:SW_CHOC_HS
- U1: footprint KBD_PARTS:ProMicro-ish-rev-unrouted_3x5 -> TB2086_MISC:ProMicro-ish-dn-rev-unrouted_3x5; symbol KBD_PARTS:ProMicro-ish -> TB2086_MISC:ProMicro-ish
Connections:
- net DATA: now also JP9.1 (A)
- net GND: now also L1.3 (VSS), L10.3 (VSS), L11.3 (VSS), L12.3 (VSS), L13.3 (VSS), L14.3 (VSS), L15.3 (VSS), L16.3 (VSS), L17.3 (VSS), L18.3 (VSS), L2.3 (VSS), L3.3 (VSS), L4.3 (VSS), L5.3 (VSS), L6.3 (VSS), L7.3 (VSS), L8.3 (VSS), L9.3 (VSS), J1.C; no longer L1.2 (VSS), L10.2 (VSS), L11.2 (VSS), L12.2 (VSS), L13.2 (VSS), L14.2 (VSS), L15.2 (VSS), L16.2 (VSS), L17.2 (VSS), L18.2 (VSS), L2.2 (VSS), L3.2 (VSS), L4.2 (VSS), L5.2 (VSS), L6.2 (VSS), L7.2 (VSS), L8.2 (VSS), L9.2 (VSS)
- net SCL: now also J1.A, R3.1
- net SDA: now also JP9.3 (B), R4.2
- net VCC: now also L1.1 (VDD), L10.1 (VDD), L11.1 (VDD), L12.1 (VDD), L13.1 (VDD), L14.1 (VDD), L15.1 (VDD), L16.1 (VDD), L17.1 (VDD), L18.1 (VDD), L2.1 (VDD), L3.1 (VDD), L4.1 (VDD), L5.1 (VDD), L6.1 (VDD), L7.1 (VDD), L8.1 (VDD), L9.1 (VDD), J1.D, R3.2, R4.1; no longer L1.4 (VDD), L10.4 (VDD), L11.4 (VDD), L12.4 (VDD), L13.4 (VDD), L14.4 (VDD), L15.4 (VDD), L16.4 (VDD), L17.4 (VDD), L18.4 (VDD), L2.4 (VDD), L3.4 (VDD), L4.4 (VDD), L5.4 (VDD), L6.4 (VDD), L7.4 (VDD), L8.4 (VDD), L9.4 (VDD)
- net at L24.1 (DOUT): now also L18.4 (DIN); no longer L18.3 (DIN)
- new net: L15.4 (DIN), L18.2 (DOUT)
- new net: L3.4 (DIN), L8.2 (DOUT)
- new net: L13.2 (DOUT), L8.4 (DIN)
- new net: L14.2 (DOUT), L17.4 (DIN)
- new net: L14.4 (DIN), L9.2 (DOUT)
- new net: L4.2 (DOUT), L9.4 (DIN)
- new net: L4.4 (DIN), L5.2 (DOUT)
- new net: L11.2 (DOUT), L6.4 (DIN)
- new net: L11.4 (DIN), L12.2 (DOUT)
- new net: J1.B, JP9.2 (C)
- new net: L13.4 (DIN), L16.2 (DOUT)
- new net: L16.4 (DIN), L17.2 (DOUT)
- new net: L2.4 (DIN), L3.2 (DOUT)
- new net: L10.2 (DOUT), L5.4 (DIN)
- new net: L2.2 (DOUT), L7.4 (DIN)
- new net: L10.4 (DIN), L15.2 (DOUT)
- new net: L1.4 (DIN), L6.2 (DOUT)
- new net: L12.4 (DIN), L7.2 (DOUT)
- no-connect marks 7 -> 6

Commit message: small tweak
Changed lines of the file:
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@@
   (symbol (lib_id "Jumper:Jumper_3_Bridged12") (at 135.255 134.62 270) (mirror x) (unit 1)
     (in_bom yes) (on_board yes) (dnp no)
-    (property "Reference" "JP9" (at 113.03 134.62 90)
+    (property "Reference" "JP9" (at 140.335 132.715 90)
       (effects (font (size 1.27 1.27)))
     )
-    (property "Value" "Jumper_3_Bridged12" (at 120.65 137.16 90)
+    (property "Value" "Jumper_3_Bridged12" (at 147.955 135.255 90)
       (effects (font (size 1.27 1.27)))
     )
