File: uniCorne-3x5/cherry-mx-reversible/unicorne-3x5-cherry-mx-reversible.kicad_pcb (KiCad board)
At the start: 2 copper layers, 114.7 x 91.4 mm, 87 parts, among them J1 MJ-4PP-9, J2 Nice!View, J3 Conn_01x02, J4 Conn_01x03, SW1 SW_MX_HS, SW10 SW_MX_HS, SW11 SW_MX_HS, SW12 SW_MX_HS, SW13 SW_MX_HS, SW14 SW_MX_HS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

Commit message: fixed 3x5
Parts:
- added JP10: Jumper_3_Bridged12, TB2086_MISC:SolderJumper-3_P1.3mm_Bridged2Bar12_RoundedPad1.0x1.5mm_rev, F.Cu at (188.3, 110.8)
- added JP11: , TB2086_MISC:SolderJumper-2_P1.3mm_Open_TrianglePad1.0x1.2mm_rev, F.Cu at (175.4, 68.8)
- JP9: value Jumper_3_Bridged12 -> (none); footprint TB2086_MISC:SolderJumper-3_P1.3mm_Bridged2Bar12_RoundedPad1.0x1.5mm_rev -> TB2086_MISC:SolderJumper-2_P1.3mm_Open_TrianglePad1.0x1.2mm_rev
- U1: footprint TB2086_MISC:ProMicro-ish-dn-rev-unrouted_3x6 -> TB2086_MISC:ProMicro-ish-dn-rev-unrouted_3x5
- moved JP9 7.39 mm to (181.7, 113.9), turned to 90 degrees
- moved R3 0.41 mm to (184.6, 110.2)
- moved R4 0.40 mm to (184.6, 112.1)
Connections:
- J1 pad A: SCL -> Net-(JP9-B)
- J1 pad B: Net-(JP9-C) -> Net-(JP10-C)
- JP9 pad 1: DATA -> SCL
- JP9 pad 2: Net-(JP9-C) -> Net-(JP9-B)
- U1 pad 24: unconnected-(U1-RAW-Pad24) -> BAT+
- U1 pad 26: GND -> B-/D-
Routing:
- net B-/D-: track 0.00 -> 18.9 mm, vias 0 -> 2
- net GND: track 38.3 -> 23.2 mm, vias 12 -> 11
- net Net-(JP9-C): track 14.5 -> 0.00 mm
- net Net-(JP10-C): track 0.00 -> 14.5 mm
- net unconnected-(U1-RAW-Pad24): track 11.0 -> 0.00 mm, vias 1 -> 0
- net Net-(JP9-B): track 0.00 -> 6.97 mm
- net BAT+: track 14.2 -> 19.8 mm
- net SCL: track 63.6 -> 61.4 mm, vias 3 -> 4
- net col1: track 152.5 -> 151.2 mm
- net col2: track 167.0 -> 165.8 mm
- net VCC: track 529.3 -> 528.0 mm
- net col3: track 142.1 -> 140.9 mm
- net col0: track 177.2 -> 177.8 mm
- net row3: track 115.6 -> 116.2 mm

Commit message: fixed 3x6
Parts:
- moved JP11 3.08 mm to (172.9, 67.0), turned to -90 degrees
Routing:
- net B-/D-: track 18.9 -> 20.9 mm
- net col0: track 177.8 -> 175.9 mm
- net GND: track 23.2 -> 24.6 mm, vias 11 -> 12
