File: uniCorne-3x5/cherry-mx-reversible/unicorne-3x5-cherry-mx-reversible.kicad_pcb (KiCad board)
At the start: 2 copper layers, 114.7 x 91.4 mm, 89 parts, among them J1 MJ-4PP-9, J2 Nice!View, J3 Conn_01x02, J4 Conn_01x03, SW1 SW_MX_HS, SW10 SW_MX_HS, SW11 SW_MX_HS, SW12 SW_MX_HS, SW13 SW_MX_HS, SW14 SW_MX_HS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

Commit message: KiCAD 8
Parts:
- D1, D10, D11, D12, D13, D15, D16, D17, D18, D2, D3, D4, D5, D6, D7, D8, D9: moved to F.Cu
- JP1, JP11, JP2, JP3, JP4, JP5, JP6, JP7, JP8, JP9: value (none) -> ~
Routing:
- net unconnected-(PSW1-C-Pad3)_1: track 5.31 -> 2.65 mm
- net unconnected-(PSW1-C-Pad3): track 0.00 -> 2.66 mm

Commit message: fixed SDA/SCL shorted
Routing:
- net unconnected-(PSW1-C-Pad3): track 2.66 -> 0.00 mm
- net unconnected-(PSW1-C-Pad3)_1: track 2.65 -> 0.00 mm
- net BAT+: vias 0 -> 1
