File: uniCorne-3x5/chocolate-reversible/unicorne-3x5-chocolate-reversible.kicad_pcb (KiCad board)
At the start: 2 copper layers, 114.7 x 91.4 mm, 89 parts, among them J1 MJ-4PP-9, J2 Conn_01x05, J3 Conn_01x02, J4 Conn_01x03, SW1 SW_CHOC_HS, SW10 SW_CHOC_HS, SW11 SW_CHOC_HS, SW12 SW_CHOC_HS, SW13 SW_CHOC_HS, SW14 SW_CHOC_HS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

Commit message: fixed 3x6
Parts:
- moved JP11 3.15 mm to (172.9, 67.0), turned to -90 degrees
Routing:
- net GND: track 31.1 -> 24.3 mm
- net row0: track 148.1 -> 144.8 mm
- net col3: track 175.9 -> 174.4 mm
- net col0: track 204.5 -> 203.1 mm
- net col1: track 186.9 -> 185.5 mm
- net col2: track 194.2 -> 193.0 mm
- net B-/D-: track 19.2 -> 20.4 mm
