File: uniCorne-3x5/chocolate-reversible/unicorne-3x5-chocolate-reversible.kicad_pcb (KiCad board)
At the start: 2 copper layers, 114.7 x 91.4 mm, 89 parts, among them J1 MJ-4PP-9, J2 Conn_01x05, J3 Conn_01x02, J4 Conn_01x03, SW1 SW_CHOC_HS, SW10 SW_CHOC_HS, SW11 SW_CHOC_HS, SW12 SW_CHOC_HS, SW13 SW_CHOC_HS, SW14 SW_CHOC_HS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

Commit message: KiCAD 8
Parts:
- D1, D10, D11, D12, D13, D14, D15, D16, D17, D18, D2, D3, D4, D5, D6, D8, D9: moved to F.Cu

Commit message: fixed SDA/SCL shorted
Routing:
- net unconnected-(PSW1-C-Pad3): vias 0 -> 1
- net BAT+: vias 0 -> 1
