File: uniCorne-3x6/hybrid-mx-reversible/unicorne-3x6-hybrid-mx-reversible.kicad_pcb (KiCad board)
At the start: 2 copper layers, 133.8 x 91.4 mm, 100 parts, among them J1 MJ-4PP-9, J2 Nice!View, J3 Conn_01x02, J4 Conn_01x03, SW1 SW_MX_HS, SW10 SW_MX_HS, SW11 SW_MX_HS, SW12 SW_MX_HS, SW13 SW_MX_HS, SW14 SW_MX_HS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

Commit message: added more docs
Parts:
- D13, D14: moved to F.Cu
