File: uniCorne-3x6/hybrid-mx-reversible/unicorne-3x6-hybrid-mx-reversible.kicad_pcb (KiCad board)
At the start: 2 copper layers, 133.8 x 91.4 mm, 98 parts, among them J1 MJ-4PP-9, J2 Nice!View, J3 Conn_01x02, J4 Conn_01x03, SW1 SW_MX_HS, SW10 SW_MX_HS, SW11 SW_MX_HS, SW12 SW_MX_HS, SW13 SW_MX_HS, SW14 SW_MX_HS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

Commit message: fixed 3x6
Parts:
- added JP10: Jumper_3_Bridged12, TB2086_MISC:SolderJumper-3_P1.3mm_Bridged2Bar12_RoundedPad1.0x1.5mm_rev, F.Cu at (188.6, 111.0)
- added JP11: , TB2086_MISC:SolderJumper-2_P1.3mm_Open_TrianglePad1.0x1.2mm_rev, F.Cu at (172.9, 67.1)
- JP9: value Jumper_3_Bridged12 -> (none); footprint TB2086_MISC:SolderJumper-3_P1.3mm_Bridged2Bar12_RoundedPad1.0x1.5mm_rev -> TB2086_MISC:SolderJumper-2_P1.3mm_Open_TrianglePad1.0x1.2mm_rev
- moved JP9 7.73 mm to (181.6, 114.0), turned to 90 degrees
- moved R4 0.50 mm to (184.9, 112.3)
- moved R3 0.47 mm to (184.9, 110.3)
Connections:
- J1 pad A: SCL -> Net-(JP9-B)
- J1 pad B: Net-(JP9-C) -> Net-(JP10-C)
- JP9 pad 1: DATA -> SCL
- JP9 pad 2: Net-(JP9-C) -> Net-(JP9-B)
- U1 pad 24: unconnected-(U1-RAW-Pad24) -> BAT+
- U1 pad 26: GND -> B-/D-
Routing:
- net B-/D-: track 0.00 -> 20.8 mm, vias 0 -> 2
- net Net-(JP9-C): track 13.9 -> 0.00 mm
- net Net-(JP10-C): track 0.00 -> 13.9 mm
- net GND: track 35.9 -> 22.6 mm, vias 17 -> 21
- net unconnected-(U1-RAW-Pad24): track 11.0 -> 0.00 mm, vias 1 -> 0
- net Net-(JP9-B): track 0.00 -> 6.84 mm
- net BAT+: track 14.2 -> 19.8 mm
- net VCC: track 577.9 -> 580.3 mm
- net SCL: track 56.8 -> 55.4 mm, vias 4 -> 5
- net col0: track 192.3 -> 191.2 mm
- net col1: track 169.2 -> 168.3 mm
- net col2: track 150.6 -> 149.7 mm
- net SDA: track 63.9 -> 63.0 mm
- net col3: track 181.9 -> 181.1 mm
- net row3: track 86.6 -> 87.2 mm
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
Commit message: Docs / KiCad8 (#12)
* KiCAD 8

* KiCad8 for plates

* Update Footprints

* Update README.md

* added more docs
Parts:
- D1, D10, D11, D12, D13, D14, D15, D16, D17, D18, D19, D2, D20, D21, D3, D4, D5, D6, D7, D8, D9: moved to F.Cu

Commit message: fixed SDA/SCL shorted
Routing:
- net unconnected-(PSW1-C-Pad3): vias 0 -> 1
- net BAT+: vias 0 -> 1
