File: case/plate/3x6/unicorne-3x6-top-plate-hybrid/unicorne-3x6-top-plate-hybrid.kicad_pcb (KiCad board)
At the start: 2 copper layers, 113 x 66 mm, 24 parts, among them SW1 SW_MX_HS, SW10 SW_MX_HS, SW11 SW_MX_HS, SW12 SW_MX_HS, SW13 SW_MX_HS, SW14 SW_MX_HS, SW15 SW_MX_HS, SW2 SW_MX_HS, SW3 SW_MX_HS, SW4 SW_MX_HS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

Commit message: fix typo
Other:
- board text added: "top plate for uniCorne hybrid designed by Allen"
- board text removed: "top plate for uniCorn hybrid designed by Allen"
