File: uniCorne-3x6/cherry-mx-reversible/unicorne-3x6-cherry-mx-reversible.kicad_pcb (KiCad board)
At the start: 2 copper layers, 133.8 x 91.4 mm, 100 parts, among them J1 MJ-4PP-9, J2 Nice!View, J3 Conn_01x02, J4 Conn_01x03, SW1 SW_MX_HS, SW10 SW_MX_HS, SW11 SW_MX_HS, SW12 SW_MX_HS, SW13 SW_MX_HS, SW14 SW_MX_HS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

Commit message: Docs / KiCad8 (#12)
* KiCAD 8

* KiCad8 for plates

* Update Footprints

* Update README.md

* added more docs
Parts:
- D1, D10, D11, D12, D13, D14, D15, D16, D17, D18, D19, D2, D20, D21, D3, D4, D5, D6, D7, D8, D9: moved to F.Cu
