File: uniCorne-3x6/cherry-mx-reversible/unicorne-3x6-cherry-mx-reversible.kicad_pcb (KiCad board)
At the start: 2 copper layers, 133.8 x 91.4 mm, 98 parts, among them J1 MJ-4PP-9, J2 Nice!View, J3 Conn_01x02, J4 Conn_01x03, SW1 SW_MX_HS, SW10 SW_MX_HS, SW11 SW_MX_HS, SW12 SW_MX_HS, SW13 SW_MX_HS, SW14 SW_MX_HS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

Commit message: fixed 3x6
Parts:
- added JP10: , TB2086_MISC:SolderJumper-2_P1.3mm_Open_TrianglePad1.0x1.2mm_rev, F.Cu at (181.6, 114.1)
- added JP11: , TB2086_MISC:SolderJumper-2_P1.3mm_Open_TrianglePad1.0x1.2mm_rev, F.Cu at (173.0, 67.0)
Connections:
- J1 pad A: SCL -> Net-(JP10-B)
- U1 pad 24: unconnected-(U1-RAW-Pad24) -> BAT+
- U1 pad 26: GND -> B-/D-
Routing:
- net B-/D-: track 0.00 -> 20.8 mm, vias 0 -> 2
- net GND: track 38.2 -> 24.5 mm, vias 15 -> 17
- net unconnected-(U1-RAW-Pad24): track 10.9 -> 0.00 mm, vias 1 -> 0
- net Net-(JP10-B): track 0.00 -> 6.74 mm
- net BAT+: track 14.0 -> 19.5 mm
- net SCL: track 58.6 -> 56.0 mm, vias 4 -> 5
- net row3: track 115.1 -> 117.4 mm
- net col4: track 146.1 -> 145.0 mm
- net col2: track 159.1 -> 158.1 mm
- net col0: track 195.2 -> 194.3 mm
- net col1: track 173.1 -> 172.1 mm
- net col3: track 168.9 -> 168.2 mm

Commit message: Update Footprints
Parts:
- D1, D10, D11, D12, D13, D14, D15, D16, D17, D18, D19, D2, D20, D21, D3, D4, D5, D6, D7, D9: moved to F.Cu

Commit message: added more docs
Parts:
- D8: moved to F.Cu

Commit message: fixed SDA/SCL shorted
Routing:
- net unconnected-(PSW1-C-Pad3)_2: vias 0 -> 1
- net BAT+: vias 0 -> 1
