File: uniCorne-3x6/cherry-mx-reversible/unicorne-3x6-cherry-mx-reversible.kicad_sch (KiCad schematic)
At the start: 98 parts, among them J1 MJ-4PP-9, J2 Nice!View, J3 Conn_01x02, J3 Conn_01x03, SW1 SW_MX_HS, SW10 SW_MX_HS, SW11 SW_MX_HS, SW12 SW_MX_HS, SW13 SW_MX_HS, SW14 SW_MX_HS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

Commit message: small tweak
Parts:
- U1: footprint TB2086_MISC:ProMicro-ish-dn-rev-unrouted_3x5 -> TB2086_MISC:ProMicro-ish-dn-rev-unrouted_3x6
Connections:
- net BAT+: now also PSW1.1 (A); no longer PSW1.3 (C)
Changed lines of the file:
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@@
   (no_connect (at 36.83 52.07))
   (no_connect (at 80.645 26.67))
-  (no_connect (at 59.69 203.835))
+  (no_connect (at 59.69 208.915))
   (no_connect (at 229.87 226.695))
   (no_connect (at 80.645 52.07))
@@
     (stroke (width 0) (type default))
   )
-  (wire (pts (xy 44.45 206.375) (xy 44.45 203.835))
+  (wire (pts (xy 44.45 211.455) (xy 44.45 203.835))
     (stroke (width 0) (type default))
   )
@@
     (stroke (width 0) (type default))
   )
-  (wire (pts (xy 44.45 206.375) (xy 46.99 206.375))
+  (wire (pts (xy 44.45 211.455) (xy 46.99 211.455))
     (stroke (width 0) (type default))
   )
@@
     (stroke (width 0) (type default))
   )
-  (wire (pts (xy 59.69 203.835) (xy 57.15 203.835))
+  (wire (pts (xy 59.69 208.915) (xy 57.15 208.915))
     (stroke (width 0) (type default))
   )
@@
     (stroke (width 0) (type default))
   )
-  (wire (pts (xy 57.15 208.915) (xy 60.325 208.915))
+  (wire (pts (xy 57.15 213.995) (xy 60.325 213.995))
     (stroke (width 0) (type default))
   )
@@
     )
   )
-  (global_label "BAT+" (shape input) (at 60.325 208.915 0) (fields_autoplaced)
+  (global_label "BAT+" (shape input) (at 60.325 213.995 0) (fields_autoplaced)
     (effects (font (size 1.1938 1.1938)) (justify left))
-    (property "Intersheetrefs" "${INTERSHEET_REFS}" (at 67.6608 208.915 0)
+    (property "Intersheetrefs" "${INTERSHEET_REFS}" (at 67.6608 213.995 0)
       (effects (font (size 1.27 1.27)) (justify left) hide)
     )
@@
     )
   )
-  (symbol (lib_id "Switch:SW_SPDT") (at 52.07 206.375 0) (unit 1)
+  (symbol (lib_id "Switch:SW_SPDT") (at 52.07 211.455 0) (mirror x) (unit 1)
     (in_bom yes) (on_board yes) (dnp no)
-    (property "Reference" "PSW1" (at 53.34 213.995 0)
-      (effects (font (size 1.27 1.27)) hide)
-    )
-    (property "Value" "SW_SPDT" (at 52.07 211.455 0)
-      (effects (font (size 1.27 1.27)))
-    )
-    (property "Footprint" "TB2086_SMD:SW_SPDT_PCM12_reversible" (at 52.07 206.375 0)
-      (effects (font (size 1.27 1.27)) hide)
-    )
-    (property "Datasheet" "~" (at 52.07 206.375 0)
+    (property "Reference" "PSW1" (at 53.34 203.835 0)
+      (effects (font (size 1.27 1.27)) hide)
+    )
+    (property "Value" "SW_SPDT" (at 52.07 217.17 0)
+      (effects (font (size 1.27 1.27)))
+    )
+    (property "Footprint" "TB2086_SMD:SW_SPDT_PCM12_reversible" (at 52.07 211.455 0)
+      (effects (font (size 1.27 1.27)) hide)
+    )
+    (property "Datasheet" "~" (at 52.07 211.455 0)
       (effects (font (size 1.27 1.27)) hide)
     )
@@
       (effects (font (size 1.524 1.524)))
     )
-    (property "Footprint" "TB2086_MISC:ProMicro-ish-dn-rev-unrouted_3x5" (at 60.325 62.865 0)
+    (property "Footprint" "TB2086_MISC:ProMicro-ish-dn-rev-unrouted_3x6" (at 60.325 62.865 0)
       (effects (font (size 1.524 1.524)))
     )

Commit message: fixed footprint for promicro-ish 3x6
Connections:
- net CS: now also U1.12 (B5); no longer U1.13 (B6)
- net IS_LEFT: now also U1.13 (B6); no longer U1.12 (B5)
Changed lines of the file:
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@@
     )
   )
-  (global_label "CS" (shape input) (at 80.645 54.61 0) (fields_autoplaced)
+  (global_label "IS_LEFT" (shape input) (at 80.645 54.61 0) (fields_autoplaced)
     (effects (font (size 1.1938 1.1938)) (justify left))
-    (property "Intersheetrefs" "${INTERSHEET_REFS}" (at 85.7069 54.61 0)
+    (property "Intersheetrefs" "${INTERSHEET_REFS}" (at 89.9706 54.61 0)
       (effects (font (size 1.27 1.27)) (justify left) hide)
     )
@@
     )
   )
-  (global_label "IS_LEFT" (shape input) (at 36.83 54.61 180) (fields_autoplaced)
+  (global_label "CS" (shape input) (at 36.83 54.61 180) (fields_autoplaced)
     (effects (font (size 1.1938 1.1938)) (justify right))
-    (property "Intersheetrefs" "${INTERSHEET_REFS}" (at 27.5044 54.61 0)
+    (property "Intersheetrefs" "${INTERSHEET_REFS}" (at 31.7681 54.61 0)
       (effects (font (size 1.27 1.27)) (justify right) hide)
     )

Commit message: fixed 3x6
Parts:
- added JP10, JP11: (no value), TB2086_MISC:SolderJumper-2_P1.3mm_Open_TrianglePad1.0x1.2mm_rev, symbol Jumper:Jumper_2_Open
Connections:
- net BAT+: now also U1.24 (RAW)
- net GND: now also JP11.2 (B); no longer U1.26 (GND)
- net SCL: now also JP10.1 (A); no longer J1.A
- new net: J1.A, JP10.2 (B)
- new net B-/D-: JP11.1 (A), U1.26 (B-/D-)
- no-connect marks 5 -> 4
Changed lines of the file:
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@@
   (junction (at 361.95 198.12) (diameter 0) (color 0 0 0 0)
   )
-  (junction (at 39.37 31.75) (diameter 0) (color 0 0 0 0)
-  )
   (junction (at 53.975 129.54) (diameter 0) (color 0 0 0 0)
   )
@@
   )
   (no_connect (at 36.83 52.07))
-  (no_connect (at 80.645 26.67))
   (no_connect (at 59.69 208.915))
   (no_connect (at 229.87 226.695))
@@
     (stroke (width 0) (type default))
   )
-  (wire (pts (xy 125.73 135.255) (xy 173.99 135.255))
+  (wire (pts (xy 125.73 135.255) (xy 134.493 135.255))
     (stroke (width 0) (type default))
   )
@@
     (stroke (width 0) (type default))
   )
+  (wire (pts (xy 144.653 135.255) (xy 173.99 135.255))
+    (stroke (width 0) (type default))
+  )
   (wire (pts (xy 318.77 109.22) (xy 318.77 113.03))
     (stroke (width 0) (type default))
@@
     (stroke (width 0) (type default))
   )
+  (wire (pts (xy 163.322 184.531) (xy 170.815 184.531))
+    (stroke (width 0) (type default))
+  )
   (wire (pts (xy 237.49 217.17) (xy 251.46 217.17))
     (stroke (width 0) (type default))
@@
     (stroke (width 0) (type default))
   )
-  (wire (pts (xy 39.37 24.13) (xy 39.37 31.75))
-    (stroke (width 0) (type default))
-  )
   (wire (pts (xy 278.13 95.885) (xy 271.145 95.885))
     (stroke (width 0) (type default))
@@
     (stroke (width 0) (type default))
   )
-  (wire (pts (xy 42.545 24.13) (xy 39.37 24.13))
+  (wire (pts (xy 42.545 24.13) (xy 36.83 24.13))
     (stroke (width 0) (type default))
   )
@@
     (stroke (width 0) (type default))
   )
+  (wire (pts (xy 141.605 187.071) (xy 141.605 184.531))
+    (stroke (width 0) (type default))
+  )
   (wire (pts (xy 50.165 121.285) (xy 50.165 141.605))
     (stroke (width 0) (type default))
@@
   )
   (wire (pts (xy 128.27 136.525) (xy 128.27 133.985))
+    (stroke (width 0) (type default))
+  )
+  (wire (pts (xy 141.605 184.531) (xy 153.162 184.531))
     (stroke (width 0) (type default))
   )
@@
     (property "Intersheetrefs" "${INTERSHEET_REFS}" (at 177.8 31.5838 90)
       (effects (font (size 1.27 1.27)) (justify left) hide)
+    )
+  )
+  (global_label "B-{slash}D-" (shape input) (at 36.83 24.13 180) (fields_autoplaced)
+    (effects (font (size 1.1938 1.1938)) (justify right))
+    (property "Intersheetrefs" "${INTERSHEET_REFS}" (at 27.4301 24.13 0)
+      (effects (font (size 1.27 1.27)) (justify right) hide)
     )
   )
@@
     )
   )
+  (global_label "BAT+" (shape input) (at 80.645 26.67 0) (fields_autoplaced)
+    (effects (font (size 1.1938 1.1938)) (justify left))
+    (property "Intersheetrefs" "${INTERSHEET_REFS}" (at 87.9808 26.67 0)
+      (effects (font (size 1.27 1.27)) (justify left) hide)
+    )
+  )
   (global_label "SCL" (shape input) (at 36.83 39.37 180) (fields_autoplaced)
     (effects (font (size 1.1938 1.1938)) (justify right))
@@
     )
   )
+  (global_label "B-{slash}D-" (shape input) (at 170.815 184.531 0) (fields_autoplaced)
+    (effects (font (size 1.1938 1.1938)) (justify left))
+    (property "Intersheetrefs" "${INTERSHEET_REFS}" (at 180.2149 184.531 0)
+      (effects (font (size 1.27 1.27)) (justify left) hide)
+    )
+  )
   (global_label "IS_LEFT" (shape input) (at 76.2 70.485 0) (fields_autoplaced)
     (effects (font (size 1.1938 1.1938)) (justify left))
@@
     )
   )
+  (symbol (lib_id "power:GND") (at 141.605 187.071 0) (mirror y) (unit 1)
+    (in_bom yes) (on_board yes) (dnp no)
+    (property "Reference" "#PWR011" (at 141.605 193.421 0)
+      (effects (font (size 1.27 1.27)) hide)
+    )
+    (property "Value" "GND" (at 141.732 191.008 0)
+      (effects (font (size 1.27 1.27)))
+    )
+    (property "Footprint" "" (at 141.605 187.071 0)
+      (effects (font (size 1.27 1.27)) hide)
+    )
+    (property "Datasheet" "" (at 141.605 187.071 0)
+      (effects (font (size 1.27 1.27)) hide)
+    )
+    (pin "1")
+    (instances
+      (project "unicorne-3x6-cherry-mx-reversible"
+        (path "/ea5c1f8d-7557-4cbf-a5a2-ee0a51c138e9"
+          (reference "#PWR011") (unit 1)
+        )
+      )
+    )
+  )
   (symbol (lib_id "Jumper:Jumper_2_Open") (at 64.77 133.985 180) (unit 1)
     (in_bom yes) (on_board yes) (dnp no)
@@
     )
     (property "Footprint" "TB2086_MISC:ProMicro-ish-dn-rev-unrouted_3x6" (at 60.325 62.865 0)
-      (effects (font (size 1.524 1.524)))
+      (effects (font (size 1.524 1.524)) hide)
     )
     (property "Datasheet" "" (at 62.865 72.39 0)
@@
     )
   )
+  (symbol (lib_id "Jumper:Jumper_2_Open") (at 139.573 135.255 0) (mirror y) (unit 1)
+    (in_bom yes) (on_board yes) (dnp no)
+    (property "Reference" "JP10" (at 139.573 133.223 0)
+      (effects (font (size 1.27 1.27)))
+    )
+    (property "Value" " " (at 139.319 136.779 0)
+      (effects (font (size 1.27 1.27)))
+    )
+    (property "Footprint" "TB2086_MISC:SolderJumper-2_P1.3mm_Open_TrianglePad1.0x1.2mm_rev" (at 139.573 135.255 0)
+      (effects (font (size 1.27 1.27)) hide)
+    )
+    (property "Datasheet" "~" (at 139.573 135.255 0)
+      (effects (font (size 1.27 1.27)) hide)
+    )
+    (pin "1")
+    (pin "2")
+    (instances
+      (project "unicorne-3x6-cherry-mx-reversible"
+        (path "/ea5c1f8d-7557-4cbf-a5a2-ee0a51c138e9"
+          (reference "JP10") (unit 1)
+        )
+      )
+    )
+  )
   (symbol (lib_id "Jumper:Jumper_2_Open") (at 64.77 175.26 180) (unit 1)
     (in_bom yes) (on_board yes) (dnp no)
@@
         )
       )
+    )
+  )
+  (symbol (lib_id "Jumper:Jumper_2_Open") (at 158.242 184.531 0) (mirror y) (unit 1)
+    (in_bom yes) (on_board yes) (dnp no)
+    (property "Reference" "JP11" (at 158.242 182.499 0)
+      (effects (font (size 1.27 1.27)))
+    )
+    (property "Value" " " (at 157.988 186.055 0)
+      (effects (font (size 1.27 1.27)))
+    )
+    (property "Footprint" "TB2086_MISC:SolderJumper-2_P1.3mm_Open_TrianglePad1.0x1.2mm_rev" (at 158.242 184.531 0)
+      (effects (font (size 1.27 1.27)) hide)
+    )
+    (property "Datasheet" "~" (at 158.242 184.531 0)
+      (effects (font (size 1.27 1.27)) hide)
+    )
+    (pin "1")
+    (pin "2")
+    (instances
+      (project "unicorne-3x6-cherry-mx-reversible"
+        (path "/ea5c1f8d-7557-4cbf-a5a2-ee0a51c138e9"
+          (reference "JP11") (unit 1)
+        )
+      )

Commit message: Docs / KiCad8 (#12)
* KiCAD 8

* KiCad8 for plates

* Update Footprints

* Update README.md

* added more docs
Parts:
- JP10, JP11, JP2, JP4, JP5, JP6, JP7, JP9: value (none) -> (none)
